File: schematic/EMeter.kicad_sch (KiCad schematic)
At the start: 7 parts, among them J1 Conn_01x01_Female, J2 Conn_01x01_Female, U1 ACS37800KMACTR-030B3-I2C

Commit message: Added the ACS37800 Power Monitoring IC
Parts:
- removed U?: STM32G071KxT, Package_QFP:LQFP-32_7x7mm_P0.8mm, symbol MCU_ST_STM32G0:STM32G071KxT
- added J3, J4: Conn_01x01_Female, symbol Connector:Conn_01x01_Female
- added R3, R4, R5, R6: 1M, symbol Device:R
- added R7: R, symbol Device:R
Connections:
- net GND: now also U1.15 (VINN), R5.2, R7.2
- net IP+: now reaches J1.1 (Pin_1), U1.1 (IP+), U1.2 (IP+), U1.3 (IP+), U1.4 (IP+)
- net IP+: now also R4.2
- net VINP: now reaches U1.16 (VINP)
- net VINP: now also R3.1, R7.1
- net IP-: now reaches U1.5 (IP-), U1.6 (IP-), U1.7 (IP-), U1.8 (IP-)
- net IP-: now also J4.1 (Pin_1); no longer J2.1 (Pin_1)
- new net: R3.2, R4.1
- new net: R5.1, R6.1
- new net N: J2.1 (Pin_1), J3.1 (Pin_1), R6.2
Other:
- note added: "Voltage Measurement"
